File: Rough Draft.kicad_sch (KiCad schematic)
At the start: 57 parts, among them J1 External Microphone, J2 Stereo Output, SW1 RotaryEncoder, SW2 RotaryEncoder, SW3 RotaryEncoder, SW4 SW_Push, SW5 SW_Push, U1 STM32F746NGHx, U2 WM8731CLSEFL, U3 CR2013-MI2120, U4 LD1117S33TR_SOT223, X3 12.288MHz

Commit message: Add files via upload
Added external oscillator, rough draft of screen circuit, switched out resistor symbols, added control circuit LED's
Parts:
- removed D1: BAT60JFILM, Diode_SMD:D_SOD-323, symbol Diode:BAT60A
- removed FB1: Ferrite Bead, Inductor_SMD:L_0805_2012Metric_Pad1.15x1.40mm_HandSolder, symbol stm32f091-rescue:Ferrite_Bead_Small-Device
- removed LD1: LED_Green, LED_SMD:LED_0805_2012Metric, symbol stm32f091-rescue:LED_Small_ALT-Device
- removed R1: 1k, Resistor_SMD:R_0805_2012Metric_Pad1.15x1.40mm_HandSolder, symbol Device:R_US
- removed U4: LD1117S33TR_SOT223, Package_TO_SOT_SMD:SOT-223-3_TabPin2, symbol Regulator_Linear:LD1117S33TR_SOT223
- added C10: .1uF, Capacitor_SMD:C_0805_2012Metric_Pad1.15x1.40mm_HandSolder, symbol Device:C
- added C11, C12: 20pF, symbol Device:C_Small
- added D1, D2, D3: LED, symbol Device:LED
- added FB1: FerriteBead, symbol Device:FerriteBead
- added IC2, IC3: 74HC245, symbol 74xx:74HC245
- added IC4: LM809, Package_TO_SOT_SMD:SOT-23, symbol Power_Supervisor:LM809
- added J3: USB_B_Mini, symbol Connector:USB_B_Mini
- added J4, J5: Conn_01x20, symbol Connector_Generic:Conn_01x20
- added Q1: BSS138, Package_TO_SOT_SMD:SOT-23, symbol Transistor_FET:BSS138
- added R10: 100K, Resistor_SMD:R_0805_2012Metric_Pad1.15x1.40mm_HandSolder, symbol Device:R_US
- added R11, R12, R14: 10K, symbol Device:R_US
- added R13: 1k, symbol Device:R_US
- added SW6: SW_Push, Button_Switch_SMD:SW_SPST_PTS645, symbol Switch:SW_Push
- added U4: LD1117S12TR_SOT223, Package_TO_SOT_SMD:SOT-223-3_TabPin2, symbol Regulator_Linear:LD1117S12TR_SOT223
- added U5, U6: 4072, symbol 4xxx:4072
- added U7: 74LVC2G32, symbol 74xGxx:74LVC2G32
- added X1: 16MHz, symbol Device:Crystal
- C1, C4: footprint Capacitor_SMD:C_0805_2012Metric_Pad1.15x1.40mm_HandSolder -> (none)
- C2, C3, C5, C6, C7, C8, C9: value .1uF -> 0.1uF; footprint Capacitor_SMD:C_0805_2012Metric_Pad1.15x1.40mm_HandSolder -> (none)
- R1, R2, R3, R36, R37, R4, R5, R6, R7, R8, R9: symbol Device:R_Small -> Device:R_US
- R33, R34, R35: symbol Device:R -> Device:R_US
Connections:
- net +3V0 is gone; now on net +3.3V: C5.1, C6.1, C7.1, C8.1
- net GND is gone; now on net +3.3V: C1.2, C2.2, C21.2, C22.1, C24.2, C25.1, C26.1, C27.1, C28.1, C3.2, C4.2, C5.2, C6.2, C7.2, C8.2, C9.2, E14.2, E15.1, E8.1, J1.S, J2.S, R35.2, R36.2, R37.2, SW1.C, SW2.C, SW3.C, U2.15 (HPGND), U2.19 (AGND), U2.25 (MODE), U2.26 (~{CSB}), U2.29 (AGND), U2.4 (DGND)
- net PA6(TIM3-CH1): now also U6.4
- net PC7(TIM3-CH2): now also U5.5
- net PD12(TIM4-CH1): now also U6.3
- net PD13(TIM1-CH2): now also U5.2
- net PE11(TIM1-CH2): now also U5.4
- net PE9(TIM1-CH1): now also U6.5
- net PF2(GPIO_Input): now also U7.2
- net PF3(GPIO_Input): now also U7.1
- net VCC: now also R8.1, SW4.2, SW5.2, IC2.20 (VCC), IC3.1 (A->B), IC3.20 (VCC), IC4.3 (VCC), J5.3 (Pin_3), R14.1; no longer R2.1, R3.1, R4.1, R5.1, R6.1, R7.1, R8.2
- net +3.3V: now reaches C3.1, C4.1
- net +3.3V: now also R8.2, R9.1, U1.C1 (VBAT), U1.E10 (VDD), U1.E7 (VDD), U1.E8 (VDD), U1.E9 (VDD), U1.F10 (VSS), U1.F11 (VDD), U1.F2 (VSS), U1.F4 (VDD), U1.F5 (VDD), U1.F6 (VSS), U1.F7 (VSS), U1.F8 (VSS), U1.F9 (VSS), U1.G10 (VSS), U1.G5 (VDD), U1.G6 (VSS), U1.H10 (VSS), U1.H11 (VDD), U1.H5 (VDD), U1.H6 (VSS), U1.J10 (VSS), U1.J11 (VDD), U1.J5 (VDD), U1.J6 (VSS), U1.K10 (VSS), U1.K11 (VDD), U1.K5 (VDD), U1.K6 (VSS), U1.K7 (VSS), U1.K8 (VSS), U1.K9 (VSS), U1.L10 (VDD), U1.L6 (VSS), U1.L7 (VDD), U1.L8 (VDD), U1.L9 (VDD), U1.M1 (VSSA), U1.R1 (VDDA), U3.1 (VCC), U3.2 (GND), C10.2, C11.1, C12.2, D1.1 (K), D2.1 (K), D3.1 (K), FB1.2, IC2.10 (GND), IC2.19 (CE), IC3.10 (GND), IC3.19 (CE), IC4.1 (GND), J3.5 (GND), J4.1 (Pin_1), J4.12 (Pin_12), J5.1 (Pin_1), J5.11 (Pin_11), R10.1, R11.2, R12.2, SW6.1, U4.1 (GND), U4.2 (VO), U5.3, U6.2
- net at U1.E6 (BOOT0): now also R11.1
- net at U1.G1 (PH0): now also C11.2, X1.2
- net at U1.H1 (PH1): now also C12.1, X1.1
- net at U1.J1 (NRST): now also C10.1, R10.2, SW6.2
- net +5V: no longer names the net of C1.1, C2.1
- net +5V: now also J3.1 (VBUS), U4.3 (VI)
- net 3VA renamed +3.3VA
- net +3.3VA: now also FB1.1
- net PC9 renamed PB12 (SPI2_NSS)
- new net: D2.2 (A), U7.7
- new net: D3.2 (A), U5.1
- new net: D1.2 (A), U6.1
- new net +VDC: J4.2 (Pin_2), J5.2 (Pin_2), R13.1
- new net CARDDET: J5.20 (Pin_20)
- new net CTP_IRQ: J4.9 (Pin_9), J5.12 (Pin_12)
- new net IM0: J5.18 (Pin_18)
- new net IM1: J5.17 (Pin_17)
- new net IM2: J5.16 (Pin_16)
- new net IM3: J5.15 (Pin_15)
- new net LCD_CS: IC3.15 (B3)
- new net LCD_CS_5V: IC3.5 (A3), J4.3 (Pin_3), J5.7 (Pin_7)
- new net LCD_DATA0: IC2.18 (B0)
- new net LCD_DATA0_5V: IC2.2 (A0), J4.13 (Pin_13)
- new net LCD_DATA1: IC2.17 (B1)
- new net LCD_DATA1_5V: IC2.3 (A1), J4.14 (Pin_14)
- new net LCD_DATA2: IC2.16 (B2)
- new net LCD_DATA2_5V: IC2.4 (A2), J4.15 (Pin_15)
- new net LCD_DATA3: IC2.15 (B3)
- new net LCD_DATA3_5V: IC2.5 (A3), J4.16 (Pin_16)
- new net LCD_DATA4: IC2.14 (B4)
- new net LCD_DATA4_5V: IC2.6 (A4), J4.17 (Pin_17)
- new net LCD_DATA5: IC2.13 (B5)
- new net LCD_DATA5_5V: IC2.7 (A5), J4.18 (Pin_18)
- new net LCD_DATA6: IC2.12 (B6)
- new net LCD_DATA6_5V: IC2.8 (A6), J4.19 (Pin_19)
- new net LCD_DATA7: IC2.11 (B7)
- new net LCD_DATA7_5V: IC2.9 (A7), J4.20 (Pin_20)
- new net LCD_LITE: J4.8 (Pin_8), J5.10 (Pin_10), R13.2
- new net LCD_RD: IC3.12 (B6)
- new net LCD_RD_5V: IC2.1 (A->B), IC3.8 (A6), J4.6 (Pin_6), R12.1
- new net LCD_RS: IC3.14 (B4)
- new net LCD_RST: IC3.11 (B7)
- new net LCD_RST_5V: IC3.9 (A7), IC4.2 (~{RESET}), J4.7 (Pin_7), J5.9 (Pin_9), R14.2
- new net LCD_RS_5V: IC3.6 (A4), J4.4 (Pin_4), J5.4 (Pin_4)
- new net LCD_WR: IC3.13 (B5)
- new net LCD_WR_5V: IC3.7 (A5), J4.5 (Pin_5), J5.8 (Pin_8)
- new net SCL_5V: J4.10 (Pin_10), J5.14 (Pin_14)
- new net SDA_5V: J4.11 (Pin_11), J5.13 (Pin_13)
- new net SDI_3V: IC3.16 (B2)
- new net SDI_5V: IC3.4 (A2), J5.6 (Pin_6)
- new net SDO: J5.5 (Pin_5)
- new net SD_CS_3V: IC3.17 (B1)
- new net SD_CS_5V: IC3.3 (A1), J5.19 (Pin_19)
Other:
- note added: "Codec Circuit"
- note added: "Control Circuit"
- note added: "Noise Circuit"
- note added: "Power Circuit"
- note removed: "(nominal: 2.95 V)"
- note removed: "2V @ 0.18mA"
- note removed: "600Ohm @ 100MHz .3 Ohm DCR, 500 mA"
- moved on the sheet: SW1, SW2, SW3, SW4, SW5

Commit message: Add files via upload
Parts:
- removed C11, C12: 20pF, symbol Device:C_Small
- removed D1, D2, D3: LED, symbol Device:LED
- removed IC2, IC3: 74HC245, symbol 74xx:74HC245
- removed IC4: LM809, Package_TO_SOT_SMD:SOT-23, symbol Power_Supervisor:LM809
- removed J4, J5: Conn_01x20, symbol Connector_Generic:Conn_01x20
- removed Q1: BSS138, Package_TO_SOT_SMD:SOT-23, symbol Transistor_FET:BSS138
- removed R11, R12, R14: 10K, symbol Device:R_US
- removed R13: 1k, symbol Device:R_US
- removed U5, U6: 4072, symbol 4xxx:4072
- removed U7: 74LVC2G32, symbol 74xGxx:74LVC2G32
- removed X1: 16MHz, symbol Device:Crystal
- R1, R2, R3, R36, R37, R4, R5, R6, R7, R8, R9: symbol Device:R_US -> Device:R_Small
- R33, R34, R35: symbol Device:R_US -> Device:R
Connections:
- net +3.3V: no longer R8.2, R9.1, U1.C1 (VBAT), U1.F10 (VSS), U1.F2 (VSS), U1.F6 (VSS), U1.F7 (VSS), U1.F8 (VSS), U1.F9 (VSS), U1.G10 (VSS), U1.G6 (VSS), U1.H10 (VSS), U1.H6 (VSS), U1.J10 (VSS), U1.J6 (VSS), U1.K10 (VSS), U1.K6 (VSS), U1.K7 (VSS), U1.K8 (VSS), U1.K9 (VSS), U1.L6 (VSS), U1.M1 (VSSA), U3.1 (VCC), U3.2 (GND), U4.1 (GND)
- net VCC: now also R2.1, R3.1, R4.1, R5.1, R6.1, R7.1, R8.2; no longer R8.1, SW4.2, SW5.2
- net NRST: now reaches C10.1, R10.2, SW6.2, U1.J1 (NRST)
- net PB12 (SPI2_NSS) renamed PC9
- new net: R8.1, SW4.2
- new net: R9.1, SW5.2
- new net: U1.F10 (VSS), U1.F2 (VSS), U1.F6 (VSS), U1.F7 (VSS), U1.F8 (VSS), U1.F9 (VSS), U1.G10 (VSS), U1.G6 (VSS), U1.H10 (VSS), U1.H6 (VSS), U1.J10 (VSS), U1.J6 (VSS), U1.K10 (VSS), U1.K6 (VSS), U1.K7 (VSS), U1.K8 (VSS), U1.K9 (VSS), U1.L6 (VSS)
Other:
- note removed: "Codec Circuit"
- note removed: "Control Circuit"
- note removed: "Noise Circuit"
- note removed: "Power Circuit"
- moved on the sheet: C1, C10, C2, C3, C4, C5, C6, C7, C8, C9, FB1, J3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
