File: Rough Draft (1).kicad_sch (KiCad schematic)
At the start: 58 parts, among them J1 External Microphone, J2 Stereo Output, J3 USB_B_Mini, SW1 RotaryEncoder, SW2 RotaryEncoder, SW3 RotaryEncoder, SW4 SW_Push, SW5 SW_Push, SW6 SW_Push, U1 STM32F746NGHx, U2 WM8731CLSEFL, U3 CR2013-MI2120, U4 LD1117S12TR_SOT223, X3 12.288MHz

Commit message: Add files via upload
Connections:
- net VCC-3.3 is gone; now on net +3.3V: C25.2, C26.2, C27.2, C28.2, E15.2, E8.2, L2.1, L2.2, R1.1, R2.1, U2.12 (HPVDD), U2.18 (AVDD), U2.3 (DCVDD), U2.5 (DBVDD)
Other:
- moved on the sheet: C5, C6, C7, C8, C9, FB1

Commit message: LCD Circuit Completed
Parts:
- removed U3: CR2013-MI2120, Display:CR2013-MI2120, symbol Driver_Display:CR2013-MI2120
- added C11, C12: 20pF, symbol Device:C_Small
- added D2, D4, D5, D6, D7: LED, symbol Device:LED
- added IC1: LM809, Package_TO_SOT_SMD:SOT-23, symbol Power_Supervisor:LM809
- added IC2, IC3: 74HC245, symbol 74xx:74HC245
- added J4, J5: Conn_01x20, symbol Connector_Generic:Conn_01x20
- added Q1, Q2, Q3: BSS138, Package_TO_SOT_SMD:SOT-23, symbol Transistor_FET:BSS138
- added R11, R14, R15: 10K, symbol Device:R_US
- added R12, R13, R16, R17, R20, R21, R26, R27: 10k, symbol Device:R_US
- added R18: 1k, symbol Device:R_US
- added R19: 2.2k, symbol Device:R_US
- added R22, R24, R25: 10, symbol Device:R_US
- added R23: 1, symbol Device:R_US
- added R28, R29, R30, R31, R32: 150, symbol Device:R_US
- added X1: 16MHz, symbol Device:Crystal
- R1, R2, R3, R36, R37, R4, R5, R6, R7, R8, R9: symbol Device:R_Small -> Device:R_US
- R33, R34, R35: symbol Device:R -> Device:R_US
Connections:
- net +3.3V: now also R8.2, R9.1, C11.1, C12.2, D2.1 (K), D4.1 (K), D5.1 (K), D6.1 (K), D7.1 (K), IC1.1 (GND), IC2.10 (GND), IC2.19 (CE), IC3.10 (GND), IC3.19 (CE), J5.17 (Pin_17), J5.18 (Pin_18), J5.19 (Pin_19), J5.20 (Pin_20), Q3.2 (S), R11.2, R15.2, R20.2, R21.2, R26.1, R27.1; no longer C25.2, C26.2, C27.2, C28.2, E15.2, E8.2, L2.1, L2.2, R1.1, R2.1, U2.12 (HPVDD), U2.18 (AVDD), U2.3 (DCVDD), U2.5 (DBVDD)
- net PC3: now also IC2.4 (A2), R28.2
- net PE11(TIM1-CH2): now also U1.R9 (PE10)
- net PE9(TIM1-CH1): now also U1.N9 (PE8)
- net VCC: now also R8.1, SW4.2, SW5.2, IC1.3 (VCC), IC2.1 (A->B), IC2.20 (VCC), IC3.20 (VCC), J5.14 (Pin_14), J5.15 (Pin_15), J5.16 (Pin_16), Q1.1 (G), Q2.1 (G), R14.1, R19.2, R22.1, R23.1, R24.1, R25.1; no longer R2.1, R3.1, R4.1, R5.1, R6.1, R7.1, R8.2
- net at U1.E6 (BOOT0): now also R11.1
- net at U1.G1 (PH0): now also C11.2, X1.2
- net at U1.H1 (PH1): now also C12.1, X1.1
- net PB10 renamed LCD_RS_5V
- net LCD_RS_5V: now also IC2.6 (A4), R29.2
- net PC6 renamed LCD_RST_5V
- net LCD_RST_5V: now also IC1.2 (~{RESET}), IC2.9 (A7), R14.2, R31.2
- net PC8 renamed LCD_WR_5V
- net LCD_WR_5V: now also IC2.7 (A5), R30.2
- net PC9 renamed LCD_CS_5V
- net LCD_CS_5V: now also IC2.5 (A3), R32.2
- new net: D2.2 (A), R30.1
- new net: Q3.1 (G), R18.2, R19.1
- new net: D7.2 (A), R32.1
- new net: D4.2 (A), R29.1
- new net: D5.2 (A), R28.1
- new net: Q1.2 (S), R13.2
- new net: Q2.3 (D), R12.2
- new net: D6.2 (A), R31.1
- new net +5V: R12.1, R13.1, R16.1, R17.1, R18.1
- new net CTP_IRQ: J5.8 (Pin_8)
- new net DB0: IC3.18 (B0), J4.7 (Pin_7)
- new net DB1: IC3.17 (B1), J4.8 (Pin_8)
- new net DB2: IC3.16 (B2), J4.9 (Pin_9)
- new net DB3: IC3.15 (B3), J4.10 (Pin_10)
- new net DB4: IC3.14 (B4), J4.11 (Pin_11)
- new net DB5: IC3.13 (B5), J4.12 (Pin_12)
- new net DB6: IC3.12 (B6), J4.13 (Pin_13)
- new net DB7: IC3.11 (B7), J4.14 (Pin_14)
- new net IM0: J5.1 (Pin_1), R27.2
- new net IM1: J5.2 (Pin_2), R26.2
- new net IM2: J5.3 (Pin_3), R21.1
- new net IM3: J5.4 (Pin_4), R20.1
- new net LCD_CS: IC2.15 (B3), J4.1 (Pin_1)
- new net LCD_DATA0_5V: IC3.2 (A0)
- new net LCD_DATA1_5V: IC3.3 (A1)
- new net LCD_DATA2_5V: IC3.4 (A2)
- new net LCD_DATA3_5V: IC3.5 (A3)
- new net LCD_DATA4_5V: IC3.6 (A4)
- new net LCD_DATA5_5V: IC3.7 (A5)
- new net LCD_DATA6_5V: IC3.8 (A6)
- new net LCD_DATA7_5V: IC3.9 (A7)
- new net LCD_RD: IC2.12 (B6), J4.4 (Pin_4)
- new net LCD_RD_5V: IC2.8 (A6), IC3.1 (A->B), R15.1
- new net LCD_RS: IC2.14 (B4), J4.2 (Pin_2)
- new net LCD_RST: IC2.11 (B7), J5.5 (Pin_5)
- new net LCD_WR: IC2.13 (B5), J4.3 (Pin_3)
- new net LEDA: J5.10 (Pin_10), J5.11 (Pin_11), J5.12 (Pin_12), J5.13 (Pin_13), R22.2, R23.2, R24.2, R25.2
- new net LEDK: J5.9 (Pin_9), Q3.3 (D)
- new net SCL_3V: J5.6 (Pin_6), Q2.2 (S), R16.2
- new net SDA_3V: J5.7 (Pin_7), Q1.3 (D), R17.2
- new net SDI: IC2.16 (B2), J4.5 (Pin_5)
- new net SDO: J4.6 (Pin_6)
- new net SD_CS_5V: IC2.3 (A1)
- new net VCC-3.3: C25.2, C26.2, C27.2, C28.2, E15.2, E8.2, L2.1, L2.2, R1.1, R2.1, U2.12 (HPVDD), U2.18 (AVDD), U2.3 (DCVDD), U2.5 (DBVDD)
Other:
- note added: "Codec Circuit"
- note added: "Control Circuit"
- note added: "LCD Circuit"
- note added: "Noise Circuit"
- note added: "Power Circuit"
- moved on the sheet: C1, C10, C2, C21, C22, C23, C24, C25, C26, C27, C28, C3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

Commit message: Updated
Parts:
- removed D4, D5, D6, D7: LED, symbol Device:LED
- removed IC1: LM809, Package_TO_SOT_SMD:SOT-23, symbol Power_Supervisor:LM809
- removed Q2, Q3: BSS138, Package_TO_SOT_SMD:SOT-23, symbol Transistor_FET:BSS138
- removed R15: 10K, symbol Device:R_US
- removed R16, R17, R20, R21, R26, R27: 10k, symbol Device:R_US
- removed R18: 1k, symbol Device:R_US
- removed R19: 2.2k, symbol Device:R_US
- removed R22, R24, R25: 10, symbol Device:R_US
- removed R23: 1, symbol Device:R_US
- removed R28, R29, R30, R31, R32: 150, symbol Device:R_US
- added D1, D3: LED, symbol Device:LED
- added IC4: LM809, Package_TO_SOT_SMD:SOT-23, symbol Power_Supervisor:LM809
- added U3: CR2013-MI2120, Display:CR2013-MI2120, symbol Driver_Display:CR2013-MI2120
- added U5, U6: 4072, symbol 4xxx:4072
- added U7: 74LVC2G32, symbol 74xGxx:74LVC2G32
- R12: value 10k -> 10K
- R13: value 10k -> 1k
Connections:
- net LEDK is gone; now on net LCD_RST_5V: J5.9 (Pin_9)
- net +3.3V: now also J4.1 (Pin_1), J4.12 (Pin_12), J5.1 (Pin_1), J5.11 (Pin_11), R12.2, D1.1 (K), D3.1 (K), IC4.1 (GND), U3.1 (VCC), U3.2 (GND), U5.3, U6.2; no longer J5.17 (Pin_17), J5.18 (Pin_18), J5.19 (Pin_19), J5.20 (Pin_20)
- net CTP_IRQ: now also J4.9 (Pin_9), J5.12 (Pin_12); no longer J5.8 (Pin_8)
- net IM0: now also J5.18 (Pin_18); no longer J5.1 (Pin_1)
- net IM1: now also J5.17 (Pin_17); no longer J5.2 (Pin_2)
- net IM2: now also J5.16 (Pin_16); no longer J5.3 (Pin_3)
- net IM3: now also J5.15 (Pin_15); no longer J5.4 (Pin_4)
- net LCD_CS: now also IC3.15 (B3); no longer IC2.15 (B3), J4.1 (Pin_1)
- net LCD_CS_5V: now also IC3.5 (A3), J4.3 (Pin_3), J5.7 (Pin_7); no longer IC2.5 (A3), U1.F14 (PC9)
- net LCD_DATA0_5V: now also IC2.2 (A0), J4.13 (Pin_13); no longer IC3.2 (A0)
- net LCD_DATA1_5V: now also IC2.3 (A1), J4.14 (Pin_14); no longer IC3.3 (A1)
- net LCD_DATA2_5V: now also IC2.4 (A2), J4.15 (Pin_15); no longer IC3.4 (A2)
- net LCD_DATA3_5V: now also IC2.5 (A3), J4.16 (Pin_16); no longer IC3.5 (A3)
- net LCD_DATA4_5V: now also IC2.6 (A4), J4.17 (Pin_17); no longer IC3.6 (A4)
- net LCD_DATA5_5V: now also IC2.7 (A5), J4.18 (Pin_18); no longer IC3.7 (A5)
- net LCD_DATA6_5V: now also IC2.8 (A6), J4.19 (Pin_19); no longer IC3.8 (A6)
- net LCD_DATA7_5V: now also IC2.9 (A7), J4.20 (Pin_20); no longer IC3.9 (A7)
- net LCD_RD: now also IC3.12 (B6); no longer IC2.12 (B6), J4.4 (Pin_4)
- net LCD_RD_5V: now also IC2.1 (A->B), IC3.8 (A6), J4.6 (Pin_6), R12.1; no longer IC2.8 (A6), IC3.1 (A->B)
- net LCD_RS: now also IC3.14 (B4); no longer IC2.14 (B4), J4.2 (Pin_2)
- net LCD_RST: now also IC3.11 (B7); no longer IC2.11 (B7), J5.5 (Pin_5)
- net LCD_RST_5V: now also IC3.9 (A7), J4.7 (Pin_7), IC4.2 (~{RESET}); no longer IC2.9 (A7), U1.H15 (PC6)
- net LCD_RS_5V: now also IC3.6 (A4), J4.4 (Pin_4), J5.4 (Pin_4); no longer IC2.6 (A4), U1.P12 (PB10)
- net LCD_WR: now also IC3.13 (B5); no longer IC2.13 (B5), J4.3 (Pin_3)
- net LCD_WR_5V: now also IC3.7 (A5), J4.5 (Pin_5), J5.8 (Pin_8); no longer IC2.7 (A5), U1.G14 (PC8)
- net PA6(TIM3-CH1): now also U6.4
- net PC3: now also U3.6 (MOSI); no longer IC2.4 (A2)
- net PC7(TIM3-CH2): now also U5.5
- net PD12(TIM4-CH1): now also U6.3
- net PD13(TIM1-CH2): now also U5.2
- net PE11(TIM1-CH2): now also U5.4; no longer U1.R9 (PE10)
- net PE9(TIM1-CH1): now also U6.5; no longer U1.N9 (PE8)
- net PF2(GPIO_Input): now also U7.2
- net PF3(GPIO_Input): now also U7.1
- net SCL_5V: now also J4.10 (Pin_10), J5.14 (Pin_14)
- net SDA_5V: now also J4.11 (Pin_11), J5.13 (Pin_13)
- net SDO: now also J5.5 (Pin_5); no longer J4.6 (Pin_6)
- net SD_CS_3V: now also IC3.17 (B1)
- net SD_CS_5V: now also IC3.3 (A1), J5.19 (Pin_19); no longer IC2.3 (A1)
- net VCC: now also IC3.1 (A->B), J5.3 (Pin_3), IC4.3 (VCC); no longer IC2.1 (A->B), J5.14 (Pin_14), J5.15 (Pin_15), J5.16 (Pin_16), Q1.1 (G)
- net at D2.2 (A): now also U7.7
- net at Q1.2 (S): no longer R13.2
- net LCD_DATA1: now reaches IC2.17 (B1)
- net LCD_DATA0: now reaches IC2.18 (B0)
- net +5V renamed +VDC
- net +VDC: now also J4.2 (Pin_2), J5.2 (Pin_2); no longer R12.1
- net DB0: no longer names the net of IC3.18 (B0)
- net DB0: no longer J4.7 (Pin_7)
- net DB1 renamed LCD_LITE
- net LCD_LITE: now also J5.10 (Pin_10), R13.2; no longer IC3.17 (B1)
- net DB2 renamed SDI_3V
- net SDI_3V: no longer J4.9 (Pin_9)
- removed net DB3: IC3.15 (B3), J4.10 (Pin_10)
- removed net DB4: IC3.14 (B4), J4.11 (Pin_11)
- removed net DB5: IC3.13 (B5), J4.12 (Pin_12)
- removed net DB6: IC3.12 (B6), J4.13 (Pin_13)
- removed net DB7: IC3.11 (B7), J4.14 (Pin_14)
- removed net LEDA: J5.10 (Pin_10), J5.11 (Pin_11), J5.12 (Pin_12), J5.13 (Pin_13)
- net SCL_3V renamed SDI_5V
- net SDI_5V: now also IC3.4 (A2)
- net SDA_3V: no longer names the net of Q1.3 (D)
- net SDA_3V: no longer J5.7 (Pin_7)
- net SDI renamed LCD_DATA2
- net LCD_DATA2: no longer J4.5 (Pin_5)
- new net: D3.2 (A), U5.1
- new net: D1.2 (A), U6.1
- new net CARDDET: J5.20 (Pin_20)
- new net LCD_DATA3: IC2.15 (B3)
- new net LCD_DATA4: IC2.14 (B4)
- new net LCD_DATA5: IC2.13 (B5)
- new net LCD_DATA6: IC2.12 (B6)
- new net LCD_DATA7: IC2.11 (B7)
- new net PB10: U1.P12 (PB10), U3.7 (SCK)
- new net PB12 (SPI2_NSS): U1.F14 (PC9), U3.3 (~{CS})
- new net PC6: U1.H15 (PC6), U3.4 (RESET)
- new net PC8: U1.G14 (PC8), U3.5 (D/~{C})
Other:
- note removed: "LCD Circuit"
- moved on the sheet: C10, C11, C12, C21, C22, C23, C24, C25, C26, C27, C28, E10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

Commit message: Add files via upload
Parts:
- removed D1, D3: LED, symbol Device:LED
- removed FB1: FerriteBead, symbol Device:FerriteBead
- removed IC4: LM809, Package_TO_SOT_SMD:SOT-23, symbol Power_Supervisor:LM809
- removed U3: CR2013-MI2120, Display:CR2013-MI2120, symbol Driver_Display:CR2013-MI2120
- removed U5, U6: 4072, symbol 4xxx:4072
- removed U7: 74LVC2G32, symbol 74xGxx:74LVC2G32
- added C13, C14, C15, C16, C17, C18, C19, C20, C29, C30, C31, C32, C33: 0.1uF, symbol Device:C
- added D1, D3: BZX84Cxx, Package_TO_SOT_SMD:SOT-23, symbol Diode:BZX84Cxx
- added D4, D5, D6, D7: LED, symbol Device:LED
- added IC1: LM809, Package_TO_SOT_SMD:SOT-23, symbol Power_Supervisor:LM809
- added Q2, Q3: BSS138, Package_TO_SOT_SMD:SOT-23, symbol Transistor_FET:BSS138
- added R15: 10K, symbol Device:R_US
- added R16, R17, R20, R21, R26, R27: 10k, symbol Device:R_US
- added R18: 1k, symbol Device:R_US
- added R19: 2.2k, symbol Device:R_US
- added R22, R24, R25: 10, symbol Device:R_US
- added R23: 1, symbol Device:R_US
- added R28, R29, R30, R31, R32: 150, symbol Device:R_US
- added R38, R39: R_Small, symbol Device:R_US
- R12: value 10K -> 10k
- R13: value 1k -> 10k
Connections:
- net +3.3VA is gone; now on net +3.3V: C9.1
- net CARDDET is gone; now on net +3.3V: J5.20 (Pin_20)
- net LCD_DATA3 is gone; now on net LCD_CS: IC2.15 (B3)
- net LCD_DATA4 is gone; now on net LCD_RS: IC2.14 (B4)
- net LCD_DATA5 is gone; now on net LCD_WR: IC2.13 (B5)
- net LCD_DATA6 is gone; now on net LCD_RD: IC2.12 (B6)
- net LCD_DATA7 is gone; now on net LCD_RST: IC2.11 (B7)
- net PB10 is gone; now on net LCD_RS_5V: U1.P12 (PB10)
- net PB12 (SPI2_NSS) is gone; now on net LCD_CS_5V: U1.F14 (PC9)
- net PC6 is gone; now on net LCD_RST_5V: U1.H15 (PC6)
- net PC8 is gone; now on net LCD_WR_5V: U1.G14 (PC8)
- net +3.3V: now also J5.17 (Pin_17), J5.18 (Pin_18), J5.19 (Pin_19), C13.1, C13.2, C14.1, C14.2, C15.1, C15.2, C16.1, C16.2, C17.1, C17.2, C18.1, C18.2, C19.1, C19.2, C20.1, C20.2, C29.1, C29.2, C30.1, C30.2, C31.1, C31.2, C32.1, C32.2, C33.1, C33.2, D1.1 (A), D3.1 (A), D4.1 (K), D5.1 (K), D6.1 (K), D7.1 (K), IC1.1 (GND), Q3.2 (S), R15.2, R20.2, R21.2, R26.1, R27.1; no longer J4.1 (Pin_1), J4.12 (Pin_12), J5.1 (Pin_1), J5.11 (Pin_11), R12.2
- net CTP_IRQ: now also J5.8 (Pin_8); no longer J4.9 (Pin_9), J5.12 (Pin_12)
- net IM0: now also J5.1 (Pin_1), R27.2; no longer J5.18 (Pin_18)
- net IM1: now also J5.2 (Pin_2), R26.2; no longer J5.17 (Pin_17)
- net IM2: now also J5.3 (Pin_3), R21.1; no longer J5.16 (Pin_16)
- net IM3: now also J5.4 (Pin_4), R20.1; no longer J5.15 (Pin_15)
- net LCD_CS: now also J4.1 (Pin_1); no longer IC3.15 (B3)
- net LCD_CS_5V: now also IC2.5 (A3), R32.2; no longer IC3.5 (A3), J4.3 (Pin_3), J5.7 (Pin_7)
- net LCD_DATA0_5V: now also IC3.2 (A0); no longer IC2.2 (A0), J4.13 (Pin_13)
- net LCD_DATA1_5V: now also IC3.3 (A1); no longer IC2.3 (A1), J4.14 (Pin_14)
- net LCD_DATA2_5V: now also IC3.4 (A2); no longer IC2.4 (A2), J4.15 (Pin_15)
- net LCD_DATA3_5V: now also IC3.5 (A3); no longer IC2.5 (A3), J4.16 (Pin_16)
- net LCD_DATA4_5V: now also IC3.6 (A4); no longer IC2.6 (A4), J4.17 (Pin_17)
- net LCD_DATA5_5V: now also IC3.7 (A5); no longer IC2.7 (A5), J4.18 (Pin_18)
- net LCD_DATA6_5V: now also IC3.8 (A6); no longer IC2.8 (A6), J4.19 (Pin_19)
- net LCD_DATA7_5V: now also IC3.9 (A7); no longer IC2.9 (A7), J4.20 (Pin_20)
- net LCD_RD: now also J4.4 (Pin_4); no longer IC3.12 (B6)
- net LCD_RD_5V: now also IC2.8 (A6), IC3.1 (A->B), R15.1; no longer IC2.1 (A->B), IC3.8 (A6), J4.6 (Pin_6), R12.1
- net LCD_RS: now also J4.2 (Pin_2); no longer IC3.14 (B4)
- net LCD_RST: now also J5.5 (Pin_5); no longer IC3.11 (B7)
- net LCD_RST_5V: now also IC2.9 (A7), IC1.2 (~{RESET}), R31.2; no longer IC3.9 (A7), J4.7 (Pin_7), J5.9 (Pin_9)
- net LCD_RS_5V: now also IC2.6 (A4), R29.2; no longer IC3.6 (A4), J4.4 (Pin_4), J5.4 (Pin_4)
- net LCD_WR: now also J4.3 (Pin_3); no longer IC3.13 (B5)
- net LCD_WR_5V: now also IC2.7 (A5), R30.2; no longer IC3.7 (A5), J4.5 (Pin_5), J5.8 (Pin_8)
- net PC3: now also IC2.4 (A2), R28.2
- net PE11(TIM1-CH2): now also U1.R9 (PE10)
- net PE9(TIM1-CH1): now also U1.N9 (PE8)
- net SCL_5V: no longer J4.10 (Pin_10), J5.14 (Pin_14)
- net SDA_5V: no longer J4.11 (Pin_11), J5.13 (Pin_13)
- net SDO: now also J4.6 (Pin_6); no longer J5.5 (Pin_5)
- net SD_CS_3V: no longer IC3.17 (B1)
- net SD_CS_5V: now also IC2.3 (A1); no longer IC3.3 (A1), J5.19 (Pin_19)
- net VCC: now also IC2.1 (A->B), J5.14 (Pin_14), J5.15 (Pin_15), J5.16 (Pin_16), Q1.1 (G), IC1.3 (VCC), Q2.1 (G), R19.2, R22.1, R23.1, R24.1, R25.1, R38.2, R39.2; no longer IC3.1 (A->B), J5.3 (Pin_3), SW4.2, SW5.2
- net at D2.2 (A): now also R30.1
- net at Q1.2 (S): now also R13.2
- net SDA_3V: now reaches Q1.3 (D)
- net SDA_3V: now also J5.7 (Pin_7), R17.2
- net DB0: now reaches IC3.18 (B0)
- net DB0: now also J4.7 (Pin_7)
- removed net +VDC: J4.2 (Pin_2), J5.2 (Pin_2), R13.1
- net LCD_DATA0: no longer names the net of IC2.18 (B0)
- net LCD_DATA1: no longer names the net of IC2.17 (B1)
- net LCD_DATA2 renamed SDI
- net SDI: now also J4.5 (Pin_5)
- removed net LCD_LITE: J4.8 (Pin_8), J5.10 (Pin_10), R13.2
- net SDI_3V renamed DB2
- net DB2: now also J4.9 (Pin_9)
- net SDI_5V renamed SCL_3V
- net SCL_3V: now also Q2.2 (S), R16.2; no longer IC3.4 (A2)
- new net: Q3.1 (G), R18.2, R19.1
- new net: D7.2 (A), R32.1
- new net: D4.2 (A), R29.1
- new net: D1.3 (K), R38.1, SW4.2
- new net: D5.2 (A), R28.1
- new net: D3.3 (K), R39.1, SW5.2
- new net: Q2.3 (D), R12.2
- new net: D6.2 (A), R31.1
- new net +5V: R12.1, R13.1, R16.1, R17.1, R18.1
- new net DB1: IC3.17 (B1), J4.8 (Pin_8)
- new net DB3: IC3.15 (B3), J4.10 (Pin_10)
- new net DB4: IC3.14 (B4), J4.11 (Pin_11)
- new net DB5: IC3.13 (B5), J4.12 (Pin_12)
- new net DB6: IC3.12 (B6), J4.13 (Pin_13)
- new net DB7: IC3.11 (B7), J4.14 (Pin_14)
- new net LEDA: J5.10 (Pin_10), J5.11 (Pin_11), J5.12 (Pin_12), J5.13 (Pin_13), R22.2, R23.2, R24.2, R25.2
- new net LEDK: J5.9 (Pin_9), Q3.3 (D)
Other:
- note added: "LCD Circuit"
- moved on the sheet: C1, C10, C11, C12, C2, C21, C22, C23, C24, C25, C26, C27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
