File: Current.kicad_pcb (KiCad board)
At the start: 2 copper layers, 73.7 x 53.3 mm, 110 parts, among them IC1 LM809, J1 USB_OTG, Q1 BSS138, Q2 BSS138, Q3 BSS138, SW1 SW_Push, SW2 SW_Push, SW3 SW_Push, SW4 RotaryEncoder, SW5 RotaryEncoder, SW6 RotaryEncoder, U1 LD1117S12TR_SOT223, U2 STM32F746NGHx, U3 WM8731CLSEFL

Commit message: Add files via upload
Parts:
- added D10: BZX84Cxx, Package_TO_SOT_SMD:SOT-23, F.Cu at (38.9, 44.0)
- added D11: BZX84Cxx, Package_TO_SOT_SMD:SOT-23, F.Cu at (38.9, 48.5)
- added D12: BZX84Cxx, Package_TO_SOT_SMD:SOT-23, F.Cu at (38.9, 52.9)
- added D13: BZX84Cxx, Package_TO_SOT_SMD:SOT-23, F.Cu at (38.9, 57.4)
- added D8: BZX84Cxx, Package_TO_SOT_SMD:SOT-23, F.Cu at (38.9, 35.1)
- added D9: BZX84Cxx, Package_TO_SOT_SMD:SOT-23, F.Cu at (38.9, 39.5)
- added IC2: 74HC245, SN74LVC245APW:SOP65P640X120-20N, F.Cu at (46.3, 37.0)
- added IC3: 74HC245, SN74LVC245APW:SOP65P640X120-20N, F.Cu at (46.3, 45.1)
- added J2: Stereo Output, SJ1_3515_SMT_TR:CUI_SJ1-3515-SMT, F.Cu at (28.2, 33.3)
- added J3: Stereo Microphone, SJ1_3515_SMT_TR:CUI_SJ1-3515-SMT, F.Cu at (28.2, 48.3)
- added J4: External Microphone, SJ1_3515_SMT_TR:CUI_SJ1-3515-SMT, F.Cu at (28.2, 63.2)
- added J7: Conn_01x50_Pin, 50 Position FPC Connector Contacts:68715014522, F.Cu at (53.8, 29.3)
- added L1: 10uH, Inductor_SMD:L_0201_0603Metric_Pad0.64x0.40mm_HandSolder, F.Cu at (54.6, 33.8)
- added R48: 220, Resistor_SMD:R_0201_0603Metric, F.Cu at (51.9, 33.8)
- added R49: 220, Resistor_SMD:R_0201_0603Metric, F.Cu at (51.9, 35.5)
- added R50: 220, Resistor_SMD:R_0201_0603Metric, F.Cu at (51.9, 37.2)
- added R51: 220, Resistor_SMD:R_0201_0603Metric, F.Cu at (51.9, 39.0)
- added R52: 220, Resistor_SMD:R_0201_0603Metric, F.Cu at (51.9, 40.8)
- added R53: 220, Resistor_SMD:R_0201_0603Metric, F.Cu at (51.9, 42.5)
- R10, R11, R12, R13, R14, R15: value R_Small -> 1k
- R19, R20: value R_Small -> 220
Connections:
- C30 pad 2: /VCC-3.3 -> /VCCA-3.3
- C31 pad 2: /VCC-3.3 -> /VCCA-3.3
- E5 pad 2: /VCC-3.3 -> /VCCA-3.3
- R10 pad 1: unconnected-(R10-Pad1) -> VCC
- R11 pad 1: unconnected-(R11-Pad1) -> VCC
- R12 pad 1: unconnected-(R12-Pad1) -> VCC
- R13 pad 1: unconnected-(R13-Pad1) -> VCC
- R14 pad 1: unconnected-(R14-Pad1) -> VCC
- R15 pad 1: unconnected-(R15-Pad1) -> VCC
- SW4 pad A: /PE9(TIM1-CH1) -> Net-(D12-K)
- SW4 pad B: /PE11(TIM1-CH2) -> Net-(D13-K)
- SW5 pad A: /PA6(TIM3-CH1) -> Net-(D10-K)
- SW5 pad B: /PC7(TIM3-CH2) -> Net-(D11-K)
- SW6 pad A: /PD12(TIM4-CH1) -> Net-(D8-K)
- SW6 pad B: /PD13(TIM1-CH2) -> Net-(D9-K)
- U2 pad A8: unconnected-(U2-PB5-PadA8) -> /CTP_IRQ
- U2 pad B5: Net-(JP2-A) -> /SDA_5V
- U2 pad B6: Net-(JP1-A) -> /SCL_5V
- U3 pad 12: /VCC-3.3 -> /VCCA-3.3
- U3 pad 18: /VCC-3.3 -> /VCCA-3.3
